File: PBSS5480X Motor Driver/PBSS5480X_Motor_Driver.sch (KiCad schematic (older format))
At the start: 75 parts, among them P1 Digital, P10 CONN_1, P11 CONN_1, P12 ESC1_Connector, P2 Analog, P3 CONN_1, P4 CONN_1, P5 CONN_1, P6 CONN_1, P7 Shield_Connector, P8 CONN_1, P9 CONN_1, Q1 DTC114E, Q2 PBSS5480X, Q3 DTC114E, Q4 DTC114E, Q5 PBSS5480X, Q6 PBSS5480X, Q7 DTC114E, Q8 PBSS5480X

Commit message: Creating Documentation
Continue Documentation adding board assembly information
Parts:
- C1, C10, C11, C12, C13, C14, C15, C16, C17, C18, C19, C2, C20, C21, C22, C23, C24, C25, C26, C3, C4, C5, C6, C7, C8, C9: symbol C -> Device:C
- D1, D10, D2, D3, D5, D6, D7, D8, D9: symbol D -> Device:D
- D4: symbol TVS -> PBSS5480X-Motor-Driver-rescue:TVS
- P1, P2, P7: symbol CONN_15 -> PBSS5480X-Motor-Driver-rescue:CONN_15
- P10, P11, P3, P4, P5, P6, P8, P9: symbol CONN_1 -> PBSS5480X-Motor-Driver-rescue:CONN_1
- P12: symbol CONN_01X03 -> PBSS5480X-Motor-Driver-rescue:CONN_01X03
- Q1, Q3, Q4, Q7: symbol DTC114E -> PBSS5480X-Motor-Driver-rescue:DTC114E
- Q2, Q5, Q6, Q8: symbol BCX53 -> PBSS5480X-Motor-Driver-rescue:BCX53
- R1, R10, R11, R12, R13, R14, R15, R16, R17, R18, R19, R2, R3, R4, R5, R6, R7, R8, R9: symbol R -> Device:R
Connections:
- wire segments 241 -> 317
